File: pcb/power/powerPCB/powerPCB.kicad_sch (KiCad schematic)
At the start: 14 parts

Commit message: updated folders
Parts:
- removed C?: 100n, symbol Device:C_Small
- removed D?: BLUE, symbol Device:LED
- removed J?: XT60PW-F, my_foot:AMASS_XT60PW-F, symbol Connector:Conn_01x02_Female
- removed R?: 330, symbol Device:R_Small
- removed R?: 52k, symbol Device:R_Small
- removed U?: TPS563202DRLR, Package_TO_SOT_SMD:SOT-23-6, symbol my_sym:TPS563202DRLR
- added C4, C7: 22u, Capacitor_SMD:C_1210_3225Metric, symbol Device:C_Small
- added H1, H2, H3: 12V, MountingHole:MountingHole_2.2mm_M2_DIN965_Pad, symbol Mechanical:MountingHole_Pad
- added H10, H7, H8, H9: MountingHole_Pad, MountingHole:MountingHole_3.2mm_M3_DIN965_Pad, symbol Mechanical:MountingHole_Pad
- added H4, H5, H6: GND, MountingHole:MountingHole_2.2mm_M2_DIN965_Pad, symbol Mechanical:MountingHole_Pad
- added J1, J2, J3, J4: 5OUT, my_foot:PinHeader_1x02_P5.00mm, symbol Connector:Conn_01x02_Female
- added J5: 12OUT, my_foot:PinHeader_1x02_P5.00mm, symbol Connector:Conn_01x02_Female
- added R3: 11k, Resistor_SMD:R_0603_1608Metric, symbol Device:R_Small
- added R4: 15k, Resistor_SMD:R_0603_1608Metric, symbol Device:R_Small
- added R5: 220k, Resistor_SMD:R_1206_3216Metric, symbol Device:R_Small
- added SW1: SW_SPDT, my_foot:remote switch, symbol Switch:SW_SPDT
- added U1: TPS566247DRLR, Package_TO_SOT_SMD:SOT-563, symbol my_sym:TPS566247DRLR
- C1, C2: renamed from C?; footprint (none) -> Capacitor_SMD:C_1206_3216Metric
- C3: renamed from C?; footprint (none) -> Capacitor_SMD:C_0603_1608Metric
- C5, C6: renamed from C?; footprint (none) -> Capacitor_SMD:C_1210_3225Metric
- L1: renamed from L?; value 4u7 -> 2u2; footprint (none) -> Inductor_SMD:L_Wuerth_WE-PD2-Typ-XL
- R1: renamed from R?; value 10k -> 100k; footprint (none) -> Resistor_SMD:R_0603_1608Metric
- R2: renamed from R?; value 10k -> 15k; footprint (none) -> Resistor_SMD:R_0603_1608Metric
Connections:
- net +12V: now also J5.1 (Pin_1), SW1.3 (C), U1.1 (VIN)
- net +5V: now also C4.1, C7.1, J1.1 (Pin_1), J2.1 (Pin_1), J3.1 (Pin_1), J4.1 (Pin_1), R5.2
- net GND: now also C1.2, C3.2, C4.2, C7.2, H4.1, H5.1, H6.1, J1.2 (Pin_2), J2.2 (Pin_2), J3.2 (Pin_2), J4.2 (Pin_2), J5.2 (Pin_2), R3.1, R4.1, U1.3 (GND), U1.4 (AGND); no longer R2.1
- net SW: now reaches L1.1
- net SW: now also U1.2 (SW)
- net EN: now reaches R1.2
- net EN: now also R3.2, U1.5 (EN)
- net FB: now reaches R2.2
- net FB: now also R5.1, U1.6 (FB)
- new net: R2.1, R4.2
- new net 12IN: H1.1, H2.1, H3.1, SW1.2 (B)
- no-connect marks 0 -> 5
Other:
- note added: "Input Connectors"
- note added: "Power Supply - 5V"
- note added: "Screw Terminal Outputs"
- note added: "inductor peak current rating > 7.03A inductor RMS current rating > 6.007A"
- note removed: "Input Connector"
- note removed: "Power Indicator LED"
- note removed: "inductor peak current rating > 3.53A inductor RMS current rating > 3.02A"
- moved on the sheet: C1, C2, C3, C5, C6, L1, R1, R2
